File: hw/nrf52811_usb/nrf52811_usb.sch (KiCad schematic (older format))
At the start: 43 parts, among them J1 USB_A, J2 UART, J3 TC2030-CTX, J4 RP_SMA, SW1 RST, SW2 RST, U1 MIC550X, U2 FT234XD, U3 NRF52811-QFAA, Y1 32.768kHz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

Commit message: Released nrf52811_usb to oshpark :D
Parts:
- removed J2: UART, Connector_PinHeader_2.54mm:PinHeader_1x03_P2.54mm_Vertical, symbol Connector_Generic:Conn_01x03
- added TP1: TX, TestPoint:TestPoint_Pad_D1.5mm, symbol Connector:TestPoint
- added TP2: RX, TestPoint:TestPoint_Pad_D1.5mm, symbol Connector:TestPoint
- added TP3: GND, TestPoint:TestPoint_Pad_D1.5mm, symbol Connector:TestPoint
- added TP4: 3V3, TestPoint:TestPoint_Pad_D1.5mm, symbol Connector:TestPoint
- J1: footprint (none) -> alvarop:MOLEX-0480371000
Connections:
- net +3V3: now also TP4.1
- net GND: now also TP3.1
- net UART_RX: now also U3.11 (P0.09), TP2.1; no longer U3.18 (P0.15)
- net UART_TX: now also U3.10 (P0.08), TP1.1; no longer U3.17 (P0.14)
Changed lines of the file:
@@
 encoding utf-8
 Sheet 1 1
-Title "Chaac"
-Date "2019-05-23"
-Rev "2.0"
+Title "NRF52811_USB"
+Date "2019-05-24"
+Rev "1.0"
 Comp "@alvaroprieto"
 Comment1 ""
@@
 Wire Wire Line
 	2650 3050 2650 2850
-$Comp
-L power:GND #PWR010
-U 1 1 5BAB8AD3
-P 3600 1550
-F 0 "#PWR010" H 3600 1300 50  0001 C CNN
-F 1 "GND" H 3605 1377 50  0000 C CNN
-F 2 "" H 3600 1550 50  0001 C CNN
-F 3 "" H 3600 1550 50  0001 C CNN
-	1    3600 1550
-	0    -1   -1   0
-$EndComp
 NoConn ~ 14100 6700
 Text Label 850  2550 2    50   ~ 0
@@
 SWCLK
 Wire Wire Line
-	9800 4600 9800 5150
-Wire Wire Line
-	9700 4600 9700 5150
-Text Label 9700 5150 1    50   ~ 0
+	8700 3900 8150 3900
+Wire Wire Line
+	8700 3800 8150 3800
+Text Label 8150 3800 0    50   ~ 0
 UART_TX
-Text Label 9800 5150 1    50   ~ 0
+Text Label 8150 3900 0    50   ~ 0
 UART_RX
-$Comp
-L Connector_Generic:Conn_01x03 J2
-U 1 1 5C923533
-P 3300 1650
-F 0 "J2" H 3220 1967 50  0000 C CNN
-F 1 "UART" H 3220 1876 50  0000 C CNN
-F 2 "Connector_PinHeader_2.54mm:PinHeader_1x03_P2.54mm_Vertical" H 3300 1650 50  0001 C CNN
-F 3 "~" H 3300 1650 50  0001 C CNN
-	1    3300 1650
-	-1   0    0    -1
-$EndComp
-Wire Wire Line
-	3600 1550 3500 1550
-Text Label 4250 1750 2    50   ~ 0
-UART_TX
 $Comp
 L Device:C_Small C15
@@
 	5200 4500 5200 4550
 Wire Wire Line
-	3500 1750 4250 1750
-Wire Wire Line
-	3500 1650 4250 1650
-Text Label 4250 1650 2    50   ~ 0
-UART_RX
-Wire Wire Line
 	850  2550 1450 2550
 Wire Wire Line
@@
 F 0 "J1" H 1557 7717 50  0000 C CNN
 F 1 "USB_A" H 1557 7626 50  0000 C CNN
-F 2 "" H 1650 7200 50  0001 C CNN
+F 2 "alvarop:MOLEX-0480371000" H 1650 7200 50  0001 C CNN
 F 3 " ~" H 1650 7200 50  0001 C CNN
 	1    1500 7250
@@
 Wire Wire Line
 	9600 4600 9600 5150
-NoConn ~ 8700 3900
-NoConn ~ 8700 3800
+NoConn ~ 9700 4600
+NoConn ~ 9800 4600
 NoConn ~ 8700 3700
 NoConn ~ 8700 3500
@@
 Wire Wire Line
 	1400 8100 1400 8000
+$Comp
+L Connector:TestPoint TP2
+U 1 1 5D271B59
+P 7500 4650
+F 0 "TP2" V 7454 4838 50  0000 L CNN
+F 1 "RX" V 7545 4838 50  0000 L CNN
+F 2 "TestPoint:TestPoint_Pad_D1.5mm" H 7700 4650 50  0001 C CNN
+F 3 "~" H 7700 4650 50  0001 C CNN
+	1    7500 4650
+	0    1    1    0
+$EndComp
+$Comp
+L Connector:TestPoint TP1
+U 1 1 5D272E09
+P 7500 4450
+F 0 "TP1" V 7454 4638 50  0000 L CNN
+F 1 "TX" V 7545 4638 50  0000 L CNN
+F 2 "TestPoint:TestPoint_Pad_D1.5mm" H 7700 4450 50  0001 C CNN
+F 3 "~" H 7700 4450 50  0001 C CNN
+	1    7500 4450
+	0    1    1    0
+$EndComp
+$Comp
+L Connector:TestPoint TP3
+U 1 1 5D275EFD
+P 7500 4850
+F 0 "TP3" V 7454 5038 50  0000 L CNN
+F 1 "GND" V 7545 5038 50  0000 L CNN
+F 2 "TestPoint:TestPoint_Pad_D1.5mm" H 7700 4850 50  0001 C CNN
+F 3 "~" H 7700 4850 50  0001 C CNN
+	1    7500 4850
+	0    1    1    0
+$EndComp
+$Comp
+L Connector:TestPoint TP4
+U 1 1 5D275F03
+P 7500 5050
+F 0 "TP4" V 7454 5238 50  0000 L CNN
+F 1 "3V3" V 7545 5238 50  0000 L CNN
+F 2 "TestPoint:TestPoint_Pad_D1.5mm" H 7700 5050 50  0001 C CNN
+F 3 "~" H 7700 5050 50  0001 C CNN
+	1    7500 5050
+	0    1    1    0
+$EndComp
+Text Label 7100 4450 0    50   ~ 0
+UART_TX
+Wire Wire Line
+	7100 4450 7500 4450
+Text Label 7100 4650 0    50   ~ 0
+UART_RX
+Wire Wire Line
+	7100 4650 7500 4650
+$Comp
+L power:GND #PWR0101
+U 1 1 5D34C3EB
+P 7350 4850
+F 0 "#PWR0101" H 7350 4600 50  0001 C CNN
+F 1 "GND" H 7355 4677 50  0000 C CNN
+F 2 "" H 7350 4850 50  0001 C CNN
+F 3 "" H 7350 4850 50  0001 C CNN
+	1    7350 4850
+	0    1    1    0
+$EndComp
+Wire Wire Line
+	7350 4850 7500 4850
+$Comp
+L power:+3.3V #PWR0102
+U 1 1 5D3564B9
+P 7350 5050
+F 0 "#PWR0102" H 7350 4900 50  0001 C CNN
+F 1 "+3.3V" H 7365 5223 50  0000 C CNN
+F 2 "" H 7350 5050 50  0001 C CNN
+F 3 "" H 7350 5050 50  0001 C CNN
+	1    7350 5050
+	0    -1   -1   0
+$EndComp
+Wire Wire Line
+	7350 5050 7500 5050
 $EndSCHEMATC

Commit message: Updated BOM for nrf52811_usb
Parts:
- C1, C5: DKPN 490-1536-1-ND -> 311-1438-1-ND; MPN GRM188R61C105KA93D -> CC0402KRX5R5BB105
- C2, C4: DKPN (none) -> 399-7796-1-ND; MPN (none) -> C0402C470K5GACTU
- C3: DKPN (none) -> 1276-1028-1-ND; MPN (none) -> CL05B103KB5NNNC
- D1, D2, D3: DKPN (none) -> 1516-1216-1-ND; MPN (none) -> QBLP595-IG
- FB1: DKPN (none) -> 490-1006-1-ND; MPN (none) -> BLM15AG601SN1D
- J1: DKPN (none) -> WM17118-ND; MPN (none) -> 0480371000
- J4: DKPN SAM8857-ND‎ -> CONREVSMA003.062-ND; MPN ‎SMA-J-P-H-ST-EM1‎ -> CONREVSMA003.062
- R2, R6: DKPN (none) -> 311-27JRCT-ND; MPN (none) -> RC0402JR-0727RL
- R3, R4, R5: DKPN (none) -> 311-10KJRCT-ND; MPN (none) -> RC0402JR-0710KL
- U2: DKPN (none) -> FT234XD-R; MPN (none) -> 768-1178-1-ND
Changed lines of the file:
@@
 F 2 "Capacitor_SMD:C_0402_1005Metric" H 1450 2750 50  0001 C CNN
 F 3 "~" H 1450 2750 50  0001 C CNN
-F 4 "490-1536-1-ND" H -3750 1250 50  0001 C CNN "DKPN"
-F 5 "GRM188R61C105KA93D" H -3750 1250 50  0001 C CNN "MPN"
+F 4 "311-1438-1-ND" H -3750 1250 50  0001 C CNN "DKPN"
+F 5 "CC0402KRX5R5BB105" H -3750 1250 50  0001 C CNN "MPN"
 	1    1450 2750
 	1    0    0    -1
@@
 F 2 "Capacitor_SMD:C_0402_1005Metric" H 2650 2750 50  0001 C CNN
 F 3 "~" H 2650 2750 50  0001 C CNN
-F 4 "490-1536-1-ND" H -3750 1250 50  0001 C CNN "DKPN"
-F 5 "GRM188R61C105KA93D" H -3750 1250 50  0001 C CNN "MPN"
+F 4 "311-1438-1-ND" H -3750 1250 50  0001 C CNN "DKPN"
+F 5 "CC0402KRX5R5BB105" H -3750 1250 50  0001 C CNN "MPN"
 	1    2650 2750
 	1    0    0    -1
@@
 F 2 "Resistor_SMD:R_0402_1005Metric" H 5950 4500 50  0001 C CNN
 F 3 "~" H 5950 4500 50  0001 C CNN
-F 4 "" H 3700 -5700 50  0001 C CNN "DKPN"
-F 5 "" H 3700 -5700 50  0001 C CNN "MPN"
+F 4 "311-10KJRCT-ND" H 3700 -5700 50  0001 C CNN "DKPN"
+F 5 "RC0402JR-0710KL" H 3700 -5700 50  0001 C CNN "MPN"
 	1    5950 4500
 	0    -1   -1   0
@@
 F 2 "LED_SMD:LED_0402_1005Metric" H 5550 4500 50  0001 C CNN
 F 3 "~" H 5550 4500 50  0001 C CNN
-F 4 "" H 0   0   50  0001 C CNN "DKPN"
-F 5 "" H 0   0   50  0001 C CNN "MPN"
+F 4 "1516-1216-1-ND" H 0   0   50  0001 C CNN "DKPN"
+F 5 "QBLP595-IG" H 0   0   50  0001 C CNN "MPN"
 	1    5550 4500
 	1    0    0    -1
@@
 F 2 "Resistor_SMD:R_0402_1005Metric" H 5950 5000 50  0001 C CNN
 F 3 "~" H 5950 5000 50  0001 C CNN
-F 4 "" H 3700 -5200 50  0001 C CNN "DKPN"
-F 5 "" H 3700 -5200 50  0001 C CNN "MPN"
+F 4 "311-10KJRCT-ND" H 3700 -5200 50  0001 C CNN "DKPN"
+F 5 "RC0402JR-0710KL" H 3700 -5200 50  0001 C CNN "MPN"
 	1    5950 5000
 	0    -1   -1   0
@@
 F 2 "LED_SMD:LED_0402_1005Metric" H 5550 5000 50  0001 C CNN
 F 3 "~" H 5550 5000 50  0001 C CNN
-F 4 "" H 0   500 50  0001 C CNN "DKPN"
-F 5 "" H 0   500 50  0001 C CNN "MPN"
+F 4 "1516-1216-1-ND" H 0   500 50  0001 C CNN "DKPN"
+F 5 "QBLP595-IG" H 0   500 50  0001 C CNN "MPN"
 	1    5550 5000
 	1    0    0    -1
@@
 F 2 "Connector_Coaxial:SMA_Samtec_SMA-J-P-H-ST-EM1_EdgeMount" H 14200 3800 50  0001 C CNN
 F 3 " ~" H 14200 3800 50  0001 C CNN
-F 4 "SAM8857-ND‎" H 14200 3800 50  0001 C CNN "DKPN"
-F 5 " ‎SMA-J-P-H-ST-EM1‎" H 14200 3800 50  0001 C CNN "MPN"
+F 4 "CONREVSMA003.062-ND" H 14200 3800 50  0001 C CNN "DKPN"
+F 5 "CONREVSMA003.062" H 14200 3800 50  0001 C CNN "MPN"
 	1    14200 3800
 	1    0    0    -1
@@
 F 2 "alvarop:FTDI_DFN12" H 5700 6800 60  0001 C CNN
 F 3 "" H 5700 6800 60  0001 C CNN
+F 4 "FT234XD-R" H 5700 6800 50  0001 C CNN "DKPN"
+F 5 "768-1178-1-ND" H 5700 6800 50  0001 C CNN "MPN"
 	1    5700 6800
 	1    0    0    -1
@@
 F 2 "alvarop:MOLEX-0480371000" H 1650 7200 50  0001 C CNN
 F 3 " ~" H 1650 7200 50  0001 C CNN
+F 4 "WM17118-ND" H 1500 7250 50  0001 C CNN "DKPN"
+F 5 "0480371000" H 1500 7250 50  0001 C CNN "MPN"
 	1    1500 7250
 	1    0    0    -1
@@
 F 2 "Inductor_SMD:L_0402_1005Metric" V 2280 7050 50  0001 C CNN
 F 3 "~" H 2350 7050 50  0001 C CNN
+F 4 "490-1006-1-ND" H 2350 7050 50  0001 C CNN "DKPN"
+F 5 "BLM15AG601SN1D" H 2350 7050 50  0001 C CNN "MPN"
 	1    2350 7050
 	0    -1   -1   0
@@
 F 2 "Capacitor_SMD:C_0402_1005Metric" H 1950 6900 50  0001 C CNN
 F 3 "~" H 1950 6900 50  0001 C CNN
+F 4 "1276-1028-1-ND" H 1950 6900 50  0001 C CNN "DKPN"
+F 5 "CL05B103KB5NNNC" H 1950 6900 50  0001 C CNN "MPN"
 	1    1950 6900
 	1    0    0    -1
@@
 F 2 "Resistor_SMD:R_0402_1005Metric" H 4950 6700 50  0001 C CNN
 F 3 "~" H 4950 6700 50  0001 C CNN
+F 4 "311-27JRCT-ND" H 4950 6700 50  0001 C CNN "DKPN"
+F 5 "RC0402JR-0727RL" H 4950 6700 50  0001 C CNN "MPN"
 	1    4950 6700
 	0    1    1    0
@@
 F 2 "Resistor_SMD:R_0402_1005Metric" H 6450 6700 50  0001 C CNN
 F 3 "~" H 6450 6700 50  0001 C CNN
+F 4 "311-27JRCT-ND" H 6450 6700 50  0001 C CNN "DKPN"
+F 5 "RC0402JR-0727RL" H 6450 6700 50  0001 C CNN "MPN"
 	1    6450 6700
 	0    1    1    0
@@
 F 2 "Capacitor_SMD:C_0402_1005Metric" H 1850 7500 50  0001 C CNN
 F 3 "~" H 1850 7500 50  0001 C CNN
+F 4 "399-7796-1-ND" H 1850 7500 50  0001 C CNN "DKPN"
+F 5 "C0402C470K5GACTU" H 1850 7500 50  0001 C CNN "MPN"
 	1    1850 7500
 	1    0    0    -1
@@
 F 2 "Capacitor_SMD:C_0402_1005Metric" H 2150 7500 50  0001 C CNN
 F 3 "~" H 2150 7500 50  0001 C CNN
+F 4 "399-7796-1-ND" H 2150 7500 50  0001 C CNN "DKPN"
+F 5 "C0402C470K5GACTU" H 2150 7500 50  0001 C CNN "MPN"
 	1    2150 7500
 	1    0    0    -1
@@
 F 2 "Resistor_SMD:R_0402_1005Metric" H 5950 5600 50  0001 C CNN
 F 3 "~" H 5950 5600 50  0001 C CNN
-F 4 "" H 3700 -4600 50  0001 C CNN "DKPN"
-F 5 "" H 3700 -4600 50  0001 C CNN "MPN"
+F 4 "311-10KJRCT-ND" H 3700 -4600 50  0001 C CNN "DKPN"
+F 5 "RC0402JR-0710KL" H 3700 -4600 50  0001 C CNN "MPN"
 	1    5950 5600
 	0    -1   -1   0
@@
 F 2 "LED_SMD:LED_0402_1005Metric" H 5550 5600 50  0001 C CNN
 F 3 "~" H 5550 5600 50  0001 C CNN
-F 4 "" H 0   1100 50  0001 C CNN "DKPN"
-F 5 "" H 0   1100 50  0001 C CNN "MPN"
+F 4 "1516-1216-1-ND" H 0   1100 50  0001 C CNN "DKPN"
+F 5 "QBLP595-IG" H 0   1100 50  0001 C CNN "MPN"
 	1    5550 5600
 	1    0    0    -1
