File: hw/nrf52811_breakout/nrf52811_breakout.kicad_pcb (KiCad board)
At the start: 4 copper layers, 41.8 x 20.2 mm, 21 parts, among them J1 20021321-00016C4LF, J2 20021321-00016C4LF, J3 TC2030-CTX, J4 RP_SMA, U3 NRF52811-QFAA, Y1 32.768kHz, Y2 32MHz

Commit message: Finished? layout for chaac radio v1.0?
Parts:
- added REF**: OSHW-Logo2_7.3x6mm_SilkScreen, Symbol:OSHW-Logo2_7.3x6mm_SilkScreen, F.Cu at (155.5, 46.2)
- J1, J2: moved to B.Cu
- J3: moved to F.Cu
- moved J2 29.7 mm to (178.0, 40.0)
- moved C15 27.3 mm to (166.5, 33.0), turned to 90 degrees
- moved C10 26.2 mm to (163.6, 43.0)
- moved C14 26.2 mm to (164.0, 37.0)
- moved U3 26.2 mm to (168.7, 39.8)
- moved C13 26.2 mm to (169.1, 45.4)
- moved C11 26.2 mm to (160.8, 40.9)
- moved C12 26.2 mm to (161.4, 39.0)
- moved C9 26.2 mm to (162.2, 41.6)
- moved F1 26.2 mm to (172.5, 36.4)
- moved L1 26.2 mm to (162.5, 36.3)
- moved L2 26.2 mm to (162.0, 37.6)
- moved Y1 26.2 mm to (161.7, 43.7)
- moved C16 25.7 mm to (172.6, 33.0)
- moved C17 25.7 mm to (173.6, 33.0)
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Connections:
- J1 pad 1: Net-(J1-Pad1) -> /P0.26
- J1 pad 10: Net-(J1-Pad10) -> /P0.03-AIN1
- J1 pad 11: Net-(J1-Pad11) -> /P0.06
- J1 pad 12: Net-(J1-Pad12) -> /P0.05-AIN3
- J1 pad 13: Net-(J1-Pad13) -> /P0.08
- J1 pad 14: Net-(J1-Pad14) -> /P0.07
- J1 pad 15: Net-(J1-Pad15) -> /P0.10
- J1 pad 16: Net-(J1-Pad16) -> /P0.09
- J1 pad 2: Net-(J1-Pad2) -> /P0.25
- J1 pad 3: Net-(J1-Pad3) -> /P0.28-AIN4
- J1 pad 4: Net-(J1-Pad4) -> /P0.27
- J1 pad 5: Net-(J1-Pad5) -> /P0.30-AIN6
- J1 pad 6: Net-(J1-Pad6) -> /P0.29-AIN5
- J1 pad 7: Net-(J1-Pad7) -> /P0.02-AIN0
- J1 pad 8: Net-(J1-Pad8) -> /P0.31-AIN7
- J1 pad 9: Net-(J1-Pad9) -> /P0.04-AIN2
- J2 pad 10: Net-(J2-Pad10) -> /P0.17
- J2 pad 11: Net-(J2-Pad11) -> /P0.16
- J2 pad 12: Net-(J2-Pad12) -> /P0.15
- J2 pad 13: Net-(J2-Pad13) -> /P0.14
- J2 pad 14: Net-(J2-Pad14) -> /P0.13
- J2 pad 15: Net-(J2-Pad15) -> /P0.12
- J2 pad 16: Net-(J2-Pad16) -> /P0.11
- J2 pad 3: Net-(J2-Pad3) -> /P0.24
- J2 pad 4: Net-(J2-Pad4) -> /P0.23
- J2 pad 5: Net-(J2-Pad5) -> /P0.22
- J2 pad 6: Net-(J2-Pad6) -> /nRST
- J2 pad 7: Net-(J2-Pad7) -> /P0.20
- J2 pad 8: Net-(J2-Pad8) -> /P0.19
- J2 pad 9: Net-(J2-Pad9) -> /P0.18
Routing:
- net /P0.03-AIN1: track 0.00 -> 25.4 mm, vias 0 -> 1
- net /P0.05-AIN3: track 0.00 -> 24.9 mm, vias 0 -> 1
- net /P0.07: track 0.00 -> 24.3 mm, vias 0 -> 1
- net /P0.09: track 0.00 -> 23.5 mm, vias 0 -> 1
- net /P0.04-AIN2: track 0.00 -> 21.8 mm, vias 0 -> 1
- net /P0.25: track 0.00 -> 21.3 mm, vias 0 -> 1
- net GND: track 2.23 -> 23.4 mm, vias 0 -> 15
- net /P0.06: track 0.00 -> 20.7 mm, vias 0 -> 1
- net /P0.27: track 0.00 -> 20.5 mm, vias 0 -> 1
- net /nRST: track 0.00 -> 20.5 mm, vias 0 -> 2
- net /P0.29-AIN5: track 0.00 -> 20.4 mm, vias 0 -> 1
- net /P0.08: track 0.00 -> 20.3 mm, vias 0 -> 1
- net /P0.31-AIN7: track 0.00 -> 20.0 mm, vias 0 -> 1
- net /P0.10: track 0.00 -> 19.7 mm, vias 0 -> 1
- net /SWCLK: track 0.00 -> 18.4 mm, vias 0 -> 2
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- added copper zone on Power.Cu, net +3V3
- added copper zone on F.Cu, net GND
- added copper zone on GND.Cu, net GND
Other:
- board size 41.8 x 20.2 mm -> 40 x 20 mm
- board text added: "Chaac Radio v1.0 by @alvaroprieto"
- board text removed: "NRF52811_USB by @alvaroprieto"
