File: hw/chaac_radio/chaac_radio.sch (KiCad schematic (older format))
At the start: 21 parts, among them J1 20021321-00016C4LF, J2 20021321-00016C4LF, J3 TC2030-CTX, J4 RP_SMA, U3 NRF52811-QFAA, Y1 32.768kHz, Y2 32MHz

Commit message: Updated bom and matched trace for JLCPCB impedance control
Parts:
- J1, J2: DKPN (none) -> 609-3708-1-ND; MPN (none) -> 20021321-00016C4LF
Changed lines of the file:
@@
 EESchema Schematic File Version 4
-LIBS:nrf52811_breakout-cache
+LIBS:chaac_radio-cache
 EELAYER 29 0
 EELAYER END
@@
 F 2 "alvarop:20021321-00016C4LF" H 6950 1950 50  0001 C CNN
 F 3 "~" H 6950 1950 50  0001 C CNN
+F 4 "609-3708-1-ND" H 6950 1950 50  0001 C CNN "DKPN"
+F 5 "20021321-00016C4LF" H 6950 1950 50  0001 C CNN "MPN"
 	1    6950 1950
 	1    0    0    -1
@@
 F 2 "alvarop:20021321-00016C4LF" H 10750 2000 50  0001 C CNN
 F 3 "~" H 10750 2000 50  0001 C CNN
+F 4 "609-3708-1-ND" H 10750 2000 50  0001 C CNN "DKPN"
+F 5 "20021321-00016C4LF" H 10750 2000 50  0001 C CNN "MPN"
 	1    10750 2000
 	1    0    0    -1
