File: hw/chaac/chaac.sch (KiCad schematic (older format))
At the start: 57 parts, among them J1 windrain, J10 Solar Panel, J3 UART, J4 Battery, J7 AM2315, Q1 Q_PMOS_GSD, SW1 RST, SW2 RST, U1 MIC550X, U2 CHAAC_RADIO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

Commit message: Forgot to commit chaac schematic! :-/
Parts:
- removed U2: CHAAC_RADIO, alvarop:CHAAC_RADIO, symbol alvarop:CHAAC_RADIO
- added J2, J3: chaac_radio, alvarop:20021121-00016C4LF, symbol Connector_Generic:Conn_02x08_Odd_Even
- renumbered C2 to C1, C16 to C10, C25 to C11, C26 to C12, C27 to C13, C28 to C14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
