File: hw/nrf5281x_usb_lora/nrf5281x_usb_lora.sch (KiCad schematic (older format))
At the start: 35 parts, among them J1 USB_A, J3 TC2030-CTX, SW1 RST, U1 MIC550X, U2 FT234XD, U3 NRF52811-QFAA, U4 E22-X00M22S, Y1 32.768kHz

Commit message: Fix part number for U2
Parts:
- U2: DKPN FT234XD-R -> 768-1178-1-ND; MPN 768-1178-1-ND -> FT234XD-R
Changed lines of the file:
@@
 F 2 "alvarop:FTDI_DFN12" H 5700 6800 60  0001 C CNN
 F 3 "" H 5700 6800 60  0001 C CNN
-F 4 "FT234XD-R" H 5700 6800 50  0001 C CNN "DKPN"
-F 5 "768-1178-1-ND" H 5700 6800 50  0001 C CNN "MPN"
+F 4 "768-1178-1-ND" H 5700 6800 50  0001 C CNN "DKPN"
+F 5 "FT234XD-R" H 5700 6800 50  0001 C CNN "MPN"
 	1    5700 6800
 	1    0    0    -1

Commit message: Updated nrf5281x_usb_lora to be smaller
Parts:
- removed SW1: RST, alvarop:PTS645SM43SMTR92, symbol Switch:SW_Push
- J3: symbol alvarop:TC2030-CTX -> nrf5281x_usb_lora-rescue:TC2030-CTX-alvarop
- U3: footprint Package_DFN_QFN:QFN-48-1EP_6x6mm_P0.4mm_EP4.6x4.6mm -> alvarop:NRF52811-QFN48-VIAS
- Y1: footprint Crystal:Crystal_SMD_3215-2Pin_3.2x1.5mm -> alvarop:ABS05; DKPN ‎SER4084CT-ND‎ -> 535-11897-1-ND; MPN FC-135 32.7680KA-AC0 -> ABS05-32.768KHZ-9-T
Connections:
- net +3V3: now also R3.2, R4.2
- net E22_BUSY: now also U3.18 (P0.15); no longer U3.15 (P0.12)
- net E22_DIO1: now also U3.17 (P0.14); no longer U3.14 (P0.11)
- net E22_DIO2: now also U3.16 (P0.13); no longer U3.23 (P0.20)
- net E22_NRST: now also U3.19 (P0.16); no longer U3.16 (P0.13)
- net E22_NSS: now also U3.23 (P0.20); no longer U3.20 (P0.17)
- net E22_RXEN: now also U3.14 (P0.11); no longer U3.21 (P0.18)
- net E22_TXEN: now also U3.15 (P0.12); no longer U3.22 (P0.19)
- net GND: no longer D1.1 (K), D2.1 (K)
- net MISO: now also U3.20 (P0.17); no longer U3.17 (P0.14)
- net MOSI: now also U3.21 (P0.18); no longer U3.18 (P0.15)
- net SCK: now also U3.22 (P0.19); no longer U3.19 (P0.16)
- net UART_RX: now also D2.1 (K), U3.38 (P0.26); no longer U3.11 (P0.09)
- net UART_TX: now also D1.1 (K), U3.37 (P0.25); no longer U3.10 (P0.08)
- net BOOT: no longer names the net of U3.12 (P0.10)
- removed net RX_LED: R4.2, U3.38 (P0.26)
- removed net TX_LED: R3.2, U3.37 (P0.25)
- no-connect marks 25 -> 28
Changed lines of the file:
@@
 $EndComp
 $Comp
-L alvarop:TC2030-CTX J3
+L nrf5281x_usb_lora-rescue:TC2030-CTX-alvarop J3
 U 1 1 5C2FAE4C
 P 13550 6650
@@
 SWCLK
 Wire Wire Line
-	8700 3900 8150 3900
-Wire Wire Line
-	8700 3800 8150 3800
-Text Label 8150 3800 0    50   ~ 0
+	10300 2300 10300 1750
+Wire Wire Line
+	10400 2300 10400 1750
+Text Label 10400 1750 3    50   ~ 0
 UART_TX
-Text Label 8150 3900 0    50   ~ 0
+Text Label 10300 1750 3    50   ~ 0
 UART_RX
 $Comp
@@
 	0    -1   -1   0
 $EndComp
-$Comp
-L Device:LED_ALT D1
-U 1 1 5D683111
-P 5550 4500
-F 0 "D1" H 5541 4716 50  0000 C CNN
-F 1 "LED_ALT" H 5541 4625 50  0000 C CNN
-F 2 "LED_SMD:LED_0402_1005Metric" H 5550 4500 50  0001 C CNN
-F 3 "~" H 5550 4500 50  0001 C CNN
-F 4 "1516-1216-1-ND" H 0   0   50  0001 C CNN "DKPN"
-F 5 "QBLP595-IG" H 0   0   50  0001 C CNN "MPN"
-	1    5550 4500
-	1    0    0    -1
-$EndComp
 Wire Wire Line
 	5700 4500 5850 4500
 Wire Wire Line
-	6050 4500 6400 4500
-Wire Wire Line
-	5400 4500 5200 4500
-$Comp
-L power:GND #PWR014
-U 1 1 5D6FB3B3
-P 5200 4550
-F 0 "#PWR014" H 5200 4300 50  0001 C CNN
-F 1 "GND" H 5205 4377 50  0000 C CNN
-F 2 "" H 5200 4550 50  0001 C CNN
-F 3 "" H 5200 4550 50  0001 C CNN
-	1    5200 4550
-	1    0    0    -1
-$EndComp
-Text Label 6400 4500 2    50   ~ 0
-TX_LED
-Wire Wire Line
-	5200 4500 5200 4550
+	5400 4500 5000 4500
+Text Label 5000 4500 0    50   ~ 0
+UART_TX
 Wire Wire Line
 	850  2550 1450 2550
-Wire Wire Line
-	8700 4000 8150 4000
-Text Label 8150 4000 0    50   ~ 0
-BOOT
-$Comp
-L Switch:SW_Push SW1
-U 1 1 5C55D249
-P 5400 2050
-F 0 "SW1" H 5250 2150 50  0000 C CNN
-F 1 "RST" H 5550 2150 50  0000 C CNN
-F 2 "alvarop:PTS645SM43SMTR92" H 5400 2250 50  0001 C CNN
-F 3 "" H 5400 2250 50  0001 C CNN
-F 4 "CKN9112CT-ND" H -50 -1550 50  0001 C CNN "DKPN"
-F 5 "PTS645SM43SMTR92 LFS" H -50 -1550 50  0001 C CNN "MPN"
-	1    5400 2050
-	1    0    0    -1
-$EndComp
-$Comp
-L power:GND #PWR012
-U 1 1 5C55D24F
-P 5150 2100
-F 0 "#PWR012" H 5150 1850 50  0001 C CNN
-F 1 "GND" H 5155 1927 50  0000 C CNN
-F 2 "" H 5150 2100 50  0001 C CNN
-F 3 "" H 5150 2100 50  0001 C CNN
-	1    5150 2100
-	1    0    0    -1
-$EndComp
-Wire Wire Line
-	5150 2100 5150 2050
-Wire Wire Line
-	5150 2050 5200 2050
-Wire Wire Line
-	5600 2050 6000 2050
-Text Label 6000 2050 2    50   ~ 0
-BOOT
 $Comp
 L Device:R_Small R4
@@
 	0    -1   -1   0
 $EndComp
-$Comp
-L Device:LED_ALT D2
-U 1 1 5C5E373C
-P 5550 5000
-F 0 "D2" H 5541 5216 50  0000 C CNN
-F 1 "LED_ALT" H 5541 5125 50  0000 C CNN
-F 2 "LED_SMD:LED_0402_1005Metric" H 5550 5000 50  0001 C CNN
-F 3 "~" H 5550 5000 50  0001 C CNN
-F 4 "1516-1216-1-ND" H 0   500 50  0001 C CNN "DKPN"
-F 5 "QBLP595-IG" H 0   500 50  0001 C CNN "MPN"
-	1    5550 5000
-	1    0    0    -1
-$EndComp
 Wire Wire Line
 	5700 5000 5850 5000
@@
 	6050 5000 6400 5000
 Wire Wire Line
-	5400 5000 5200 5000
-$Comp
-L power:GND #PWR015
-U 1 1 5C5E3745
-P 5200 5050
-F 0 "#PWR015" H 5200 4800 50  0001 C CNN
-F 1 "GND" H 5205 4877 50  0000 C CNN
-F 2 "" H 5200 5050 50  0001 C CNN
-F 3 "" H 5200 5050 50  0001 C CNN
-	1    5200 5050
-	1    0    0    -1
-$EndComp
-Text Label 6400 5000 2    50   ~ 0
-RX_LED
-Wire Wire Line
-	5200 5000 5200 5050
+	5400 5000 5000 5000
+Text Label 5000 5000 0    50   ~ 0
+UART_RX
 $Comp
 L power:+3.3V #PWR030
@@
 	-1   0    0    1
 $EndComp
-Text Label 10300 1750 3    50   ~ 0
-RX_LED
-Wire Wire Line
-	10300 2300 10300 1750
-Wire Wire Line
-	10400 2300 10400 1750
-Text Label 10400 1750 3    50   ~ 0
-TX_LED
 Wire Wire Line
 	9200 2200 9200 2300
@@
 F 0 "Y1" V 7350 3050 50  0000 L CNN
 F 1 "32.768kHz" V 7450 3050 50  0000 L CNN
-F 2 "Crystal:Crystal_SMD_3215-2Pin_3.2x1.5mm" H 7700 3050 50  0001 C CNN
+F 2 "alvarop:ABS05" H 7700 3050 50  0001 C CNN
 F 3 "~" H 7700 3050 50  0001 C CNN
-F 4 "‎SER4084CT-ND‎" H 7700 3050 50  0001 C CNN "DKPN"
-F 5 "FC-135 32.7680KA-AC0" H 7700 3050 50  0001 C CNN "MPN"
+F 4 "535-11897-1-ND" H 7700 3050 50  0001 C CNN "DKPN"
+F 5 "ABS05-32.768KHZ-9-T" H 7700 3050 50  0001 C CNN "MPN"
 	1    7700 3050
 	0    1    1    0
@@
 F 0 "U3" H 8250 4750 60  0000 L CNN
 F 1 "NRF52811-QFAA" H 8100 4650 60  0000 L CNN
-F 2 "Package_DFN_QFN:QFN-48-1EP_6x6mm_P0.4mm_EP4.6x4.6mm" H 8700 4000 50  0001 C CNN
+F 2 "alvarop:NRF52811-QFN48-VIAS" H 8700 4000 50  0001 C CNN
 F 3 "" H 8700 4000 50  0001 C CNN
 F 4 "‎1490-1075-1-ND‎" H 9850 3450 50  0001 C CNN "DKPN"
@@
 $EndComp
 Wire Wire Line
-	10000 4600 10000 5000
+	10300 4600 10300 5000
+Wire Wire Line
+	10200 4600 10200 5000
+Wire Wire Line
+	10100 4600 10100 5000
 Wire Wire Line
 	9900 4600 9900 5000
 Wire Wire Line
 	9800 4600 9800 5000
-Wire Wire Line
-	9600 4600 9600 5000
-Wire Wire Line
-	9500 4600 9500 5000
-Wire Wire Line
-	9400 4600 9400 5000
-Text Label 9400 5000 1    50   ~ 0
-E22_DIO1
-Text Label 10000 5000 1    50   ~ 0
-E22_NSS
-Text Label 9900 5000 1    50   ~ 0
-SCK
-Text Label 9800 5000 1    50   ~ 0
-MOSI
-Text Label 9600 5000 1    50   ~ 0
-E22_NRST
-Text Label 9500 5000 1    50   ~ 0
-E22_BUSY
 Wire Wire Line
 	9700 4600 9700 5000
 Text Label 9700 5000 1    50   ~ 0
+E22_DIO1
+Text Label 10300 5000 1    50   ~ 0
+E22_NSS
+Text Label 10200 5000 1    50   ~ 0
+SCK
+Text Label 10100 5000 1    50   ~ 0
+MOSI
+Text Label 9900 5000 1    50   ~ 0
+E22_NRST
+Text Label 9800 5000 1    50   ~ 0
+E22_BUSY
+Wire Wire Line
+	10000 4600 10000 5000
+Text Label 10000 5000 1    50   ~ 0
 MISO
 Wire Wire Line
-	10100 4600 10100 5000
-Wire Wire Line
-	10200 4600 10200 5000
-Wire Wire Line
-	10300 4600 10300 5000
-Text Label 10300 5000 1    50   ~ 0
+	9400 4600 9400 5000
+Wire Wire Line
+	9500 4600 9500 5000
+Wire Wire Line
+	9600 4600 9600 5000
+Text Label 9600 5000 1    50   ~ 0
 E22_DIO2
-Text Label 10200 5000 1    50   ~ 0
+Text Label 9500 5000 1    50   ~ 0
 E22_TXEN
-Text Label 10100 5000 1    50   ~ 0
+Text Label 9400 5000 1    50   ~ 0
 E22_RXEN
 NoConn ~ 9900 6800
+$Comp
+L Device:LED_ALT D2
+U 1 1 5C5E373C
+P 5550 5000
+F 0 "D2" H 5541 5216 50  0000 C CNN
+F 1 "LED_ALT" H 5541 5125 50  0000 C CNN
+F 2 "LED_SMD:LED_0402_1005Metric" H 5550 5000 50  0001 C CNN
+F 3 "~" H 5550 5000 50  0001 C CNN
+F 4 "1516-1216-1-ND" H 0   500 50  0001 C CNN "DKPN"
+F 5 "QBLP595-IG" H 0   500 50  0001 C CNN "MPN"
+	1    5550 5000
+	1    0    0    -1
+$EndComp
+$Comp
+L Device:LED_ALT D1
+U 1 1 5D683111
+P 5550 4500
+F 0 "D1" H 5541 4716 50  0000 C CNN
+F 1 "LED_ALT" H 5541 4625 50  0000 C CNN
+F 2 "LED_SMD:LED_0402_1005Metric" H 5550 4500 50  0001 C CNN
+F 3 "~" H 5550 4500 50  0001 C CNN
+F 4 "1516-1216-1-ND" H 0   0   50  0001 C CNN "DKPN"
+F 5 "QBLP595-IG" H 0   0   50  0001 C CNN "MPN"
+	1    5550 4500
+	1    0    0    -1
+$EndComp
+Wire Wire Line
+	6050 4500 6400 4500
+$Comp
+L power:+3.3V #PWR0101
+U 1 1 5FB442BB
+P 6400 4400
+F 0 "#PWR0101" H 6400 4250 50  0001 C CNN
+F 1 "+3.3V" H 6415 4573 50  0000 C CNN
+F 2 "" H 6400 4400 50  0001 C CNN
+F 3 "" H 6400 4400 50  0001 C CNN
+	1    6400 4400
+	1    0    0    -1
+$EndComp
+Wire Wire Line
+	6400 4400 6400 4500
+$Comp
+L power:+3.3V #PWR0102
+U 1 1 5FB4EF30
+P 6400 4900
+F 0 "#PWR0102" H 6400 4750 50  0001 C CNN
+F 1 "+3.3V" H 6415 5073 50  0000 C CNN
+F 2 "" H 6400 4900 50  0001 C CNN
+F 3 "" H 6400 4900 50  0001 C CNN
+	1    6400 4900
+	1    0    0    -1
+$EndComp
+Wire Wire Line
+	6400 4900 6400 5000
+NoConn ~ 8700 3800
+NoConn ~ 8700 3900
+NoConn ~ 8700 4000
 $EndSCHEMATC
