File: hw/chaac_ng/chaac_ng.kicad_pcb (KiCad board)
At the start: 4 copper layers, 13 x 5.9 mm, 71 parts, among them J1 Battery, J2 Solar, J3 TC2030-CTX, J4 Conn_01x04, P1 USB_C_Plug_USB2.0, SW1 SW_Push, SW2 SW_Push, U1 E22-X00M22S, U2 BQ24074RGT, U3 TPS76333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

Commit message: More placement/routing
Parts:
- P1: footprint alvarop:USB4515-GF-A -> easyeda:USB-C-SMD_TYPE-C16PIN
- moved J4 113.0 mm to (90.8, 132.1)
- moved C2 102.2 mm to (96.8, 113.9), turned to 90 degrees
- moved C5 101.9 mm to (99.4, 92.8), turned to 180 degrees
- moved C1 100.2 mm to (98.7, 110.6), turned to -90 degrees
- moved R19 98.9 mm to (86.9, 101.0), turned to -90 degrees
- moved C12 96.6 mm to (88.4, 99.9), turned to 0 degrees
- moved R21 92.2 mm to (90.5, 97.5), turned to -90 degrees
- moved SW1 91.6 mm to (110.5, 85.2), turned to -90 degrees
- moved U4 91.4 mm to (87.1, 95.2), turned to -90 degrees
- moved R1 90.6 mm to (96.8, 110.6), turned to 90 degrees
- moved C14 90.6 mm to (83.6, 92.5), turned to 90 degrees
- moved R4 89.7 mm to (97.8, 113.9), turned to 90 degrees
- moved R2 89.6 mm to (97.8, 110.6), turned to -90 degrees
- moved R20 89.6 mm to (106.3, 99.0), turned to 90 degrees
- moved SW2 88.9 mm to (110.3, 96.2), turned to -90 degrees
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Connections:
- J3 pad 6: /SWO -> unconnected-(J3-SWO-Pad6)
- U5 pad 14: /RADIO_NRST -> /RS232_EN
- U5 pad 15: /RADIO_BUSY -> /NINVALID
- U5 pad 20: /LED1 -> unconnected-(U5-PA10-Pad20)
- U5 pad 21: /USB_DM -> /USB_DN
- U5 pad 26: /SWO -> /LED1
- U5 pad 29: /NINVALID -> /RADIO_NRST
- U5 pad 30: /RS232_EN -> /RADIO_BUSY
Routing:
- net GND: track 4.30 -> 44.4 mm, vias 3 -> 27
- net /RADIO_DIO1: track 0.00 -> 36.7 mm, vias 0 -> 2
- net /MISO: track 0.00 -> 32.5 mm, vias 0 -> 2
- net /MOSI: track 0.00 -> 31.8 mm, vias 0 -> 2
- net /RADIO_NRST: track 0.00 -> 31.0 mm, vias 0 -> 2
- net /RADIO_BUSY: track 0.00 -> 30.0 mm, vias 0 -> 2
- net /SCK: track 0.00 -> 29.2 mm, vias 0 -> 2
- net /RADIO_CS: track 0.00 -> 28.0 mm, vias 0 -> 2
- net /VBATT: track 4.91 -> 29.0 mm, vias 0 -> 2
- net /RADIO_DIO2: track 0.00 -> 23.2 mm, vias 0 -> 2
- net /RADIO_RXEN: track 0.00 -> 19.7 mm, vias 0 -> 2
- net /RADIO_TXEN: track 0.00 -> 18.1 mm, vias 0 -> 2
- net +3.3V: track 3.92 -> 16.2 mm, vias 0 -> 4
- net /NRST: track 0.00 -> 5.14 mm
- net Net-(D1-K): track 10.5 -> 8.54 mm
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Other:
- board outline removed

Commit message: More layout/routing
Parts:
- moved R5 10.1 mm to (106.0, 124.1), turned to 180 degrees
- moved R6 2.51 mm to (103.5, 114.5), turned to -90 degrees
- moved J4 1.92 mm to (92.1, 133.5)
- moved P1 1.63 mm to (108.0, 118.2)
- moved J2 1.57 mm to (99.0, 133.5)
- moved D1 0.28 mm to (101.3, 121.9)
Routing:
- net /USB_DP: track 0.00 -> 21.0 mm
- net /USB_DN: track 0.00 -> 20.5 mm
- net VBUS: track 0.00 -> 13.8 mm, vias 0 -> 2
- net +6V: track 0.00 -> 9.90 mm
- net Net-(D1-K): track 8.54 -> 18.1 mm
- net /SOLAR_IN: track 0.00 -> 8.76 mm
- net /VIN: track 22.6 -> 29.5 mm
- net GND: track 44.4 -> 46.7 mm, vias 27 -> 35
- net /VBATT: track 29.0 -> 30.7 mm
- added copper zone on In1.Cu, net GND
Other:
- board outline added: 32 x 64 mm

Commit message: Releaed to JLCPCB
Parts:
- removed P1: USB_C_Plug_USB2.0, easyeda:USB-C-SMD_TYPE-C16PIN
- added G***: LOGO, alvarop:weather_station_tiny, F.Cu at (108.5, 83.0)
- added G***: LOGO, alvarop:weather_station, B.Cu at (97.3, 109.4)
- added H1: MountingHole, MountingHole:MountingHole_3.2mm_M3, F.Cu at (85.0, 74.0)
- added H2: MountingHole, MountingHole:MountingHole_3.2mm_M3, F.Cu at (109.0, 74.0)
- added J5: USB_C_Receptacle_USB2.0_16P, easyeda:USB-C-SMD_TYPE-C16PIN, F.Cu at (108.0, 118.2)
- added REF**: OSHW-Logo2_7.3x6mm_SilkScreen, Symbol:OSHW-Logo2_7.3x6mm_SilkScreen, F.Cu at (85.3, 80.6)
- J2: footprint TerminalBlock_TE-Connectivity:TerminalBlock_TE_282834-2_1x02_P2.54mm_Horizontal -> alvarop:TerminalBlock_TE_282834-2_1x02_P2.54mm_Horizontal
- J4: footprint TerminalBlock_TE-Connectivity:TerminalBlock_TE_282834-4_1x04_P2.54mm_Horizontal -> alvarop:TerminalBlock_TE_282834-4_1x04_P2.54mm_Horizontal
- moved C4 17.5 mm to (86.8, 86.5), turned to -90 degrees
- moved C3 16.4 mm to (87.8, 86.5), turned to -90 degrees
- moved U1 16.1 mm to (90.0, 71.3), turned to 90 degrees
- moved SW2 5.21 mm to (110.9, 101.4), turned to 90 degrees
- moved SW1 5.20 mm to (110.9, 90.4)
- moved C14 2.69 mm to (84.7, 90.1)
- moved R21 2.41 mm to (90.3, 99.9), turned to 180 degrees
- moved D5 2.06 mm to (106.6, 105.0)
- moved R19 2.03 mm to (85.5, 99.5), turned to 180 degrees
- moved C2 1.99 mm to (98.8, 113.9), turned to -90 degrees
- moved R25 1.97 mm to (106.6, 102.5)
- moved R3 1.93 mm to (96.8, 113.9), turned to 90 degrees
- moved D6 1.51 mm to (108.2, 105.0)
- moved R27 1.44 mm to (108.2, 102.5)
- moved R6 1.06 mm to (103.5, 115.5), turned to 90 degrees
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Routing:
- net /RS232_RX: track 0.00 -> 45.7 mm, vias 0 -> 1
- net /RS232_TX: track 0.00 -> 39.6 mm, vias 0 -> 1
- net /NRST: track 5.14 -> 36.2 mm, vias 0 -> 2
- net GND: track 46.7 -> 66.9 mm, vias 35 -> 53
- net /RS232_EN: track 0.00 -> 18.4 mm, vias 0 -> 2
- net /NINVALID: track 0.00 -> 17.6 mm
- net /SOLAR: track 1.97 -> 19.3 mm, vias 0 -> 2
- net unconnected-(J5-SHIELD-PadS1): track 0.00 -> 16.9 mm
- net /RADIO_RXEN: track 19.7 -> 35.5 mm
- net /SWDIO: track 0.00 -> 14.9 mm
- net /RADIO_TXEN: track 18.1 -> 32.7 mm
- net /BATT: track 1.97 -> 15.3 mm, vias 0 -> 2
- net /RADIO_DIO2: track 23.2 -> 36.4 mm
- net /RADIO_DIO1: track 36.7 -> 23.9 mm
- net Net-(U4-ROUT): track 0.00 -> 12.7 mm
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- added copper zone on In2.Cu, net +3.3V
Other:
- board size 32 x 64 mm -> 32 x 66 mm
- board text added: "+"
- board text added: "-"
- board text added: "6V"
- board text added: "BOOT"
- board text added: "Chaac"
- board text added: "GND"
- board text added: "RST"
- board text added: "RX"
- board text added: "TX"
- board text added: "v${REVISION}"

Commit message: Chaac ng 7.1
Parts:
- added H3: MountingHole, MountingHole:MountingHole_3.2mm_M3, F.Cu at (116.5, 159.0)
- added H4: MountingHole, MountingHole:MountingHole_3.2mm_M3, F.Cu at (85.0, 159.0)
- added H5: MountingHole, alvarop:ZIPTIE_HOLE_4x2mm, F.Cu at (92.8, 151.0)
- added H6: MountingHole, alvarop:ZIPTIE_HOLE_4x2mm, F.Cu at (105.2, 151.0)
- added H7: MountingHole, alvarop:ZIPTIE_HOLE_4x2mm, F.Cu at (110.2, 151.0)
- added H8: MountingHole, alvarop:ZIPTIE_HOLE_4x2mm, F.Cu at (117.6, 151.0)
- added J6: 6V_PWR, alvarop:TerminalBlock_TE_282834-2_1x02_P2.54mm_Horizontal, F.Cu at (94.6, 132.2)
- added R28: 43k, Resistor_SMD:R_0402_1005Metric, F.Cu at (88.7, 123.7)
- J4: value Conn_01x04 -> DATA
- R23: value 715k -> 750k
- moved REF** 79.4 mm to (102.0, 158.2)
- moved G*** 22.3 mm to (86.2, 83.0)
- moved J2 16.7 mm to (115.7, 132.2)
- moved J4 14.7 mm to (106.7, 132.2)
- moved R5 10.5 mm to (109.9, 114.3)
- moved J5 8.75 mm to (115.0, 113.0)
- moved J3 8.49 mm to (115.3, 104.6)
- moved SW2 8.20 mm to (116.9, 95.8), turned to -90 degrees
- moved J1 7.83 mm to (112.2, 123.3), turned to -90 degrees
- moved R6 7.67 mm to (109.9, 111.3), turned to 180 degrees
- moved H2 7.50 mm to (116.5, 74.0)
- moved SW1 5.76 mm to (112.8, 95.8)
- moved G*** 4.07 mm to (101.4, 109.6)
- moved C3 3.96 mm to (91.8, 86.5)
- moved C4 3.96 mm to (90.8, 86.5)
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Connections:
- J4 pad 4: +6V -> unconnected-(J4-Pin_4-Pad4)
- R19 pad 2: +3.3V -> GND
- R21 pad 1: GND -> +3.3V
- R23 pad 2: Net-(U6-FB) -> Net-(R23-Pad2)
Routing:
- net VBUS: track 14.8 -> 35.1 mm
- net /SOLAR_IN: track 20.5 -> 31.5 mm
- net /RS232_RX: track 45.7 -> 52.3 mm
- net /BOOT: track 8.31 -> 14.6 mm
- net /RS232_TX: track 39.6 -> 45.2 mm
- net Net-(J5-CC1): track 7.24 -> 2.25 mm
- net /RADIO_DIO2: track 36.4 -> 32.0 mm
- net /USB_DN: track 24.6 -> 20.3 mm, vias 0 -> 2
- net /SCK: track 27.2 -> 31.2 mm
- net /RADIO_CS: track 27.9 -> 31.9 mm
- net /MISO: track 26.0 -> 30.0 mm
- net /USB_DP: track 24.5 -> 20.5 mm, vias 2 -> 0
- net /MOSI: track 27.5 -> 31.5 mm
- net /RADIO_TXEN: track 32.7 -> 28.8 mm
- net /RADIO_DIO1: track 23.9 -> 27.7 mm
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Other:
- board size 32 x 66 mm -> 39 x 92 mm
- board text added: "BLU"
- board text added: "BRN"
- board text added: "GRN"
- board text added: "RED"
- board text added: "RESET"
- board text added: "SOLAR+"
- board text added: "SOLAR-"
- board text added: "WHT"
- board text removed: "+"
- board text removed: "-"
- board text removed: "RST"

Commit message: Released v7.1 to JLCPCB
Parts:
- removed H7, H8: MountingHole, alvarop:ZIPTIE_HOLE_4x2mm
- REF**: moved to B.Cu
- SW1, SW2: footprint alvarop:PTS636_G -> easyeda:SW-SMD_L3.9-W3.0-P4.45
- moved REF** 84.4 mm to (100.3, 73.8), turned to 180 degrees
- moved J6 54.1 mm to (110.3, 80.4), turned to -90 degrees
- moved G*** 51.2 mm to (86.3, 134.2)
- moved J4 45.0 mm to (110.3, 87.3), turned to -90 degrees
- moved SW2 39.5 mm to (101.2, 132.0), turned to 90 degrees
- moved SW1 39.3 mm to (97.4, 132.0), turned to 90 degrees
- moved G*** 26.7 mm to (100.7, 136.3)
- moved H6 13.2 mm to (110.2, 138.7), turned to -90 degrees
- moved H5 12.4 mm to (90.5, 138.8), turned to -90 degrees
- moved J2 5.33 mm to (110.3, 132.0), turned to -90 degrees
- moved C3 4.00 mm to (87.8, 86.5)
- moved C4 4.00 mm to (86.8, 86.5)
- moved U1 4.00 mm to (90.0, 71.3)
- moved J3 2.74 mm to (115.4, 101.9), turned to -90 degrees
Routing:
- net +6V: track 10.1 -> 87.2 mm
- net /BOOT: track 14.6 -> 42.9 mm, vias 0 -> 2
- net /RS232_RX: track 52.3 -> 28.6 mm, vias 1 -> 0
- net /NRST: track 37.3 -> 58.8 mm, vias 2 -> 3
- net /SWDIO: track 17.5 -> 24.9 mm
- net /SWCLK: track 14.9 -> 21.5 mm
- net /RS232_TX: track 45.2 -> 38.7 mm, vias 1 -> 0
- net /RADIO_DIO1: track 27.7 -> 23.3 mm
- net /RADIO_RXEN: track 31.9 -> 36.1 mm
- net /MISO: track 30.0 -> 25.8 mm
- net /RADIO_CS: track 31.9 -> 27.9 mm
- net /SCK: track 31.2 -> 27.2 mm
- net /MOSI: track 31.5 -> 27.5 mm
- net /RADIO_TXEN: track 28.8 -> 32.8 mm
- net /RADIO_DIO2: track 32.0 -> 35.3 mm
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Other:
- outline, holes or cut-outs redrawn
- board text added: "BATTERY"
- board text added: "BL"
- board text added: "BR"
- board text added: "GN"
- board text added: "RD"
- board text added: "S+"
- board text added: "S-"
- board text added: "WH"
- board text removed: "6V"
- board text removed: "BLU"
- board text removed: "BRN"
- board text removed: "GND"
- board text removed: "GRN"
- board text removed: "RED"
- board text removed: "RX"
- board text removed: "SOLAR+"
- board text removed: "SOLAR-"
- board text removed: "TX"
- board text removed: "WHT"
