File: hw/chaac_ng/chaac_ng.kicad_sch (KiCad schematic)
At the start: 71 parts, among them J1 Battery, J2 Solar, J3 TC2030-CTX, J4 Conn_01x04, P1 USB_C_Plug_USB2.0, SW1 SW_Push, SW2 SW_Push, U1 E22-X00M22S, U2 BQ24074RGT, U3 TPS76333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

Commit message: More placement/routing
Parts:
- P1: footprint alvarop:USB4515-GF-A -> easyeda:USB-C-SMD_TYPE-C16PIN
Connections:
- net LED1: now also U5.26 (PB3); no longer U5.20 (PA10)
- net NINVALID: now also U5.15 (PB1); no longer U5.29 (PB6)
- net RADIO_BUSY: now also U5.30 (PB7); no longer U5.15 (PB1)
- net RADIO_NRST: now also U5.29 (PB6); no longer U5.14 (PB0)
- net RS232_EN: now also U5.14 (PB0); no longer U5.30 (PB7)
- net SWO: no longer names the net of J3.6 (SWO)
- net SWO: no longer U5.26 (PB3)
- net USB_DM renamed USB_DN
- no-connect marks 2 -> 4
Changed lines of the file:
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@@
   )
   (no_connect (at 30.48 68.58))
+  (no_connect (at 271.78 200.66))
   (no_connect (at 63.5 243.84))
+  (no_connect (at 271.78 149.86))
   (wire (pts (xy 66.04 215.9) (xy 66.04 218.44))
     (stroke (width 0) (type default))
@@
     (stroke (width 0) (type default))
   )
-  (wire (pts (xy 271.78 200.66) (xy 279.4 200.66))
-    (stroke (width 0) (type default))
-  )
   (wire (pts (xy 233.68 134.62) (xy 233.68 129.54))
     (stroke (width 0) (type default))
@@
     (stroke (width 0) (type default))
   )
-  (wire (pts (xy 271.78 149.86) (xy 289.56 149.86))
-    (stroke (width 0) (type default))
-  )
   (wire (pts (xy 233.68 129.54) (xy 220.98 129.54))
     (stroke (width 0) (type default))
@@
     (effects (font (size 1.27 1.27)) (justify left bottom))
   )
-  (label "RADIO_NRST" (at 228.6 142.24 0) (fields_autoplaced)
-    (effects (font (size 1.27 1.27)) (justify left bottom))
-  )
-  (label "USB_DM" (at 71.12 43.18 180) (fields_autoplaced)
+  (label "RADIO_NRST" (at 228.6 154.94 0) (fields_autoplaced)
+    (effects (font (size 1.27 1.27)) (justify left bottom))
+  )
+  (label "USB_DN" (at 71.12 43.18 180) (fields_autoplaced)
     (effects (font (size 1.27 1.27)) (justify right bottom))
   )
@@
     (effects (font (size 1.27 1.27)) (justify left bottom))
   )
-  (label "SWO" (at 279.4 200.66 180) (fields_autoplaced)
-    (effects (font (size 1.27 1.27)) (justify right bottom))
-  )
   (label "VIN" (at 154.94 76.2 0) (fields_autoplaced)
     (effects (font (size 1.27 1.27)) (justify left bottom))
@@
     (effects (font (size 1.27 1.27)) (justify left bottom))
   )
-  (label "RADIO_BUSY" (at 228.6 144.78 0) (fields_autoplaced)
+  (label "RADIO_BUSY" (at 228.6 157.48 0) (fields_autoplaced)
     (effects (font (size 1.27 1.27)) (justify left bottom))
   )
@@
     (effects (font (size 1.27 1.27)) (justify left bottom))
   )
-  (label "RS232_EN" (at 228.6 157.48 0) (fields_autoplaced)
+  (label "RS232_EN" (at 228.6 142.24 0) (fields_autoplaced)
     (effects (font (size 1.27 1.27)) (justify left bottom))
   )
@@
     (effects (font (size 1.27 1.27)) (justify right bottom))
   )
-  (label "SWO" (at 228.6 147.32 0) (fields_autoplaced)
-    (effects (font (size 1.27 1.27)) (justify left bottom))
-  )
   (label "BQ_TMR" (at 106.68 86.36 0) (fields_autoplaced)
     (effects (font (size 1.27 1.27)) (justify left bottom))
@@
     (effects (font (size 1.27 1.27)) (justify left bottom))
   )
-  (label "NINVALID" (at 228.6 154.94 0) (fields_autoplaced)
-    (effects (font (size 1.27 1.27)) (justify left bottom))
-  )
-  (label "LED1" (at 289.56 149.86 180) (fields_autoplaced)
-    (effects (font (size 1.27 1.27)) (justify right bottom))
+  (label "NINVALID" (at 228.6 144.78 0) (fields_autoplaced)
+    (effects (font (size 1.27 1.27)) (justify left bottom))
+  )
+  (label "LED1" (at 228.6 147.32 0) (fields_autoplaced)
+    (effects (font (size 1.27 1.27)) (justify left bottom))
   )
   (label "SWDIO" (at 289.56 157.48 180) (fields_autoplaced)
@@
     (effects (font (size 1.27 1.27)) (justify left bottom))
   )
-  (label "USB_DM" (at 289.56 152.4 180) (fields_autoplaced)
+  (label "USB_DN" (at 289.56 152.4 180) (fields_autoplaced)
     (effects (font (size 1.27 1.27)) (justify right bottom))
   )
@@
       (effects (font (size 1.27 1.27)))
     )
-    (property "Footprint" "alvarop:USB4515-GF-A" (at 41.91 45.72 0)
-      (effects (font (size 1.27 1.27)) hide)
-    )
+    (property "Footprint" "easyeda:USB-C-SMD_TYPE-C16PIN" (at 41.91 45.72 0)
+      (effects (font (size 1.27 1.27)) hide)
+    )

Commit message: Releaed to JLCPCB
Parts:
- removed P1: USB_C_Plug_USB2.0, easyeda:USB-C-SMD_TYPE-C16PIN, symbol Connector:USB_C_Plug_USB2.0
- added H1, H2: MountingHole, MountingHole:MountingHole_3.2mm_M3, symbol Mechanical:MountingHole
- added J5: USB_C_Receptacle_USB2.0_16P, easyeda:USB-C-SMD_TYPE-C16PIN, symbol Connector:USB_C_Receptacle_USB2.0_16P
- C1, C12, C13, C14, C17, C2, C20, C22, C4, C5, C6, C7: LCSC (none) -> C307331; MPN (none) -> CL05B104KB54PNC
- C10, C11: LCSC (none) -> C1547; MPN (none) -> 0402CG120J500NT
- C15, C3, C9: LCSC (none) -> C52923; MPN (none) -> CL05A105KA5NQNC
- C16: LCSC (none) -> C96446; MPN (none) -> CL10A106MA8NRNC
- C18: LCSC (none) -> C15195; MPN (none) -> CL05B103KB5NNNC
- C19, C8: LCSC (none) -> C23733; MPN (none) -> CL05A475MP5NRNC
- C21: LCSC (none) -> C1546; MPN (none) -> 0402CG101J500NT
- C23: LCSC (none) -> C386098; MPN (none) -> TMK325B7226KMHP
- D1, D2: JLCPN C483994 -> (none); LCSC (none) -> C483994
- D3, D4, D5, D6: LCSC (none) -> C2286; MPN (none) -> KT-0603R
- J1: JLCPN C295747 -> (none); LCSC (none) -> C295747
- J2: footprint TerminalBlock_TE-Connectivity:TerminalBlock_TE_282834-2_1x02_P2.54mm_Horizontal -> alvarop:TerminalBlock_TE_282834-2_1x02_P2.54mm_Horizontal; JLCPN C918120 -> (none); LCSC (none) -> C918120
- J4: footprint TerminalBlock_TE-Connectivity:TerminalBlock_TE_282834-4_1x04_P2.54mm_Horizontal -> alvarop:TerminalBlock_TE_282834-4_1x04_P2.54mm_Horizontal; JLCPN C918122 -> (none); LCSC (none) -> C918122; MPN 282834-2 -> 282834-4
- L1: JLCPN C161082 -> (none); LCSC (none) -> C161082
- R1, R2, R3, R4: LCSC (none) -> C26083
- R10, R11, R14, R15, R19, R21, R8: LCSC (none) -> C17168
- R12, R13, R16, R17, R20, R25, R27, R7: LCSC (none) -> C25744
- R18: LCSC (none) -> C25867
- R22: LCSC (none) -> C227201
- R23: LCSC (none) -> C114761
- R24: LCSC (none) -> C138046
- R26: LCSC (none) -> C227250
- R5, R6: LCSC (none) -> C25905
- R9: LCSC (none) -> C11702
- SW1, SW2: JLCPN C2689642 -> (none); LCSC (none) -> C2689642
- U1: LCSC (none) -> C411293; MPN (none) -> E22-900M22S
- U2: LCSC (none) -> C54313; MPN (none) -> BQ24074RGTR
- U3: JLCPN C146356 -> (none); LCSC (none) -> C146356
- U4: JLCPN C484736 -> (none); LCSC (none) -> C484736
- U5: JLCPN C529438 -> (none); LCSC (none) -> C529438
- U6: LCSC (none) -> C128617; MPN (none) -> TPS61252DSGR
- Y1: JLCPN C596929 -> (none); LCSC (none) -> C596929
Connections:
- net GND: now also J5.A1 (GND), J5.A12 (GND), J5.B1 (GND), J5.B12 (GND)
- net USB_DN: now also J5.A7 (D-), J5.B7 (D-)
- net USB_DP: now also J5.A6 (D+), J5.B6 (D+)
- net VBUS: now also J5.A4 (VBUS), J5.A9 (VBUS), J5.B4 (VBUS), J5.B9 (VBUS)
- net at R5.1: now also J5.A5 (CC1)
- net at R6.1: now also J5.B5 (CC2)
- no-connect marks 4 -> 6

Commit message: Chaac ng 7.1
Parts:
- added H3, H4: MountingHole, MountingHole:MountingHole_3.2mm_M3, symbol Mechanical:MountingHole
- added H5, H6, H7, H8: MountingHole, alvarop:ZIPTIE_HOLE_4x2mm, symbol Mechanical:MountingHole
- added J6: 6V_PWR, alvarop:TerminalBlock_TE_282834-2_1x02_P2.54mm_Horizontal, symbol Connector_Generic:Conn_01x02
- added R28: 43k, Resistor_SMD:R_0402_1005Metric, symbol Device:R_Small
- J4: value Conn_01x04 -> DATA
- R23: value 715k -> 750k; LCSC C114761 -> C137937
Connections:
- net +3.3V: now also R21.1; no longer R19.2
- net +6V: now also J6.2 (Pin_2); no longer J4.4 (Pin_4)
- net GND: now also R19.2, J6.1 (Pin_1); no longer R21.1
- net at C21.2, R24.1, U6.3 (FB): now also R28.2; no longer R23.2
- new net: R23.2, R28.1
- no-connect marks 6 -> 7
Other:
- company: (none) -> Quesadillon LLC
- title: (none) -> Chaac NG
- moved on the sheet: R19, R24

Commit message: Released v7.1 to JLCPCB
Parts:
- removed H7, H8: MountingHole, alvarop:ZIPTIE_HOLE_4x2mm, symbol Mechanical:MountingHole
- R28: LCSC (none) -> C227081
- SW1, SW2: footprint alvarop:PTS636_G -> easyeda:SW-SMD_L3.9-W3.0-P4.45; LCSC C2689642 -> C115357; MPN PTS636 SK25 SMTR LFS -> SKRKAEE020
Changed lines of the file:
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@@
       (effects (font (size 1.27 1.27)) hide)
     )
-    (property "LCSC" "" (at 299.72 49.53 0)
+    (property "LCSC" "C227081" (at 299.72 49.53 0)
       (effects (font (size 1.27 1.27)) hide)
     )
@@
     )
   )
-  (symbol (lib_id "Mechanical:MountingHole") (at 332.74 205.74 0) (unit 1)
-    (in_bom no) (on_board yes) (dnp yes) (fields_autoplaced)
-    (property "Reference" "H7" (at 335.28 204.47 0)
-      (effects (font (size 1.27 1.27)) (justify left))
-    )
-    (property "Value" "MountingHole" (at 335.28 207.01 0)
-      (effects (font (size 1.27 1.27)) (justify left))
-    )
-    (property "Footprint" "alvarop:ZIPTIE_HOLE_4x2mm" (at 332.74 205.74 0)
-      (effects (font (size 1.27 1.27)) hide)
-    )
-    (property "Datasheet" "~" (at 332.74 205.74 0)
-      (effects (font (size 1.27 1.27)) hide)
-    )
-    (instances
-      (project "chaac_ng"
-        (path "/28e226e6-a1fa-4960-9647-597e7aabb626"
-          (reference "H7") (unit 1)
-        )
-      )
-    )
-  )
   (symbol (lib_id "Device:C_Small") (at 281.94 96.52 0) (unit 1)
     (in_bom yes) (on_board yes) (dnp no) (fields_autoplaced)
@@
     )
   )
-  (symbol (lib_id "Mechanical:MountingHole") (at 353.06 205.74 0) (unit 1)
-    (in_bom no) (on_board yes) (dnp yes) (fields_autoplaced)
-    (property "Reference" "H8" (at 355.6 204.47 0)
-      (effects (font (size 1.27 1.27)) (justify left))
-    )
-    (property "Value" "MountingHole" (at 355.6 207.01 0)
-      (effects (font (size 1.27 1.27)) (justify left))
-    )
-    (property "Footprint" "alvarop:ZIPTIE_HOLE_4x2mm" (at 353.06 205.74 0)
-      (effects (font (size 1.27 1.27)) hide)
-    )
-    (property "Datasheet" "~" (at 353.06 205.74 0)
-      (effects (font (size 1.27 1.27)) hide)
-    )
-    (instances
-      (project "chaac_ng"
-        (path "/28e226e6-a1fa-4960-9647-597e7aabb626"
-          (reference "H8") (unit 1)
-        )
-      )
-    )
-  )
   (symbol (lib_id "power:GND") (at 33.02 185.42 0) (unit 1)
     (in_bom yes) (on_board yes) (dnp no)
@@
       (effects (font (size 1.27 1.27)) (justify left))
     )
-    (property "Footprint" "alvarop:PTS636_G" (at 187.96 139.7 0)
+    (property "Footprint" "easyeda:SW-SMD_L3.9-W3.0-P4.45" (at 187.96 139.7 0)
       (effects (font (size 1.27 1.27)) hide)
     )
@@
       (effects (font (size 1.27 1.27)) hide)
     )
-    (property "MPN" "PTS636 SK25 SMTR LFS" (at 182.88 139.7 0)
+    (property "MPN" "SKRKAEE020" (at 182.88 139.7 0)
       (effects (font (size 1.27 1.27)) hide)
     )
-    (property "LCSC" "C2689642" (at 186.69 138.43 0)
+    (property "LCSC" "C115357" (at 186.69 138.43 0)
       (effects (font (size 1.27 1.27)) hide)
     )
@@
       (effects (font (size 1.27 1.27)))
     )
-    (property "Footprint" "alvarop:PTS636_G" (at 160.02 139.7 0)
+    (property "Footprint" "easyeda:SW-SMD_L3.9-W3.0-P4.45" (at 160.02 139.7 0)
       (effects (font (size 1.27 1.27)) hide)
     )
@@
       (effects (font (size 1.27 1.27)) hide)
     )
-    (property "MPN" "PTS636 SK25 SMTR LFS" (at 165.1 139.7 0)
+    (property "MPN" "SKRKAEE020" (at 165.1 139.7 0)
       (effects (font (size 1.27 1.27)) hide)
     )
-    (property "LCSC" "C2689642" (at 157.48 139.7 0)
+    (property "LCSC" "C115357" (at 157.48 139.7 0)
       (effects (font (size 1.27 1.27)) hide)
     )
